Commit message: quadrotor with full dynamics

File: quadrotor_gym/assets/quadrotor.urdf (robot description, URDF)
Before this commit: robot quadrotor, 5 links, 4 joints
Links:
- link base_link: mass 1.0 -> 0.027; geometry collision box size=0.078 0.078 0.02; visual box size=0.078 0.078 0.02
- link rotor1: mass 0.1 -> 0.001; geometry collision cylinder length=0.005 radius=0.0225; visual cylinder length=0.005 radius=0.0225
- link rotor2: mass 0.1 -> 0.001; geometry collision cylinder length=0.005 radius=0.0225; visual cylinder length=0.005 radius=0.0225
- link rotor3: mass 0.1 -> 0.001; geometry collision cylinder length=0.005 radius=0.0225; visual cylinder length=0.005 radius=0.0225
- link rotor4: mass 0.1 -> 0.001; geometry collision cylinder length=0.005 radius=0.0225; visual cylinder length=0.005 radius=0.0225
Joints:
- joint rotor1_joint: origin xyz=0.1 0.1 0.02 -> xyz=0.039 0.039 0.02
- joint rotor2_joint: origin xyz=-0.1 0.1 0.02 -> xyz=-0.039 0.039 0.02
- joint rotor3_joint: origin xyz=-0.1 -0.1 0.02 -> xyz=-0.039 -0.039 0.02
- joint rotor4_joint: origin xyz=0.1 -0.1 0.02 -> xyz=0.039 -0.039 0.02
